File: cell-voltage-amplifier.brd (EAGLE design)
At the start: 50 x 50 mm, 44 parts, among them IC1 AS321, IC10 AS321, IC2 AS321, IC3 AS321, IC4 AS321, IC7 AS321, IC9 AS321, X1 B7B-XH-2, X2 B8B-XH-2, X3 B8B-XH-2

Commit message: Done Routing
Parts:
- added C4: (no value), EcoCar-Passives:0805
- moved C2 1.59 mm to (21.0, 47.9)
- moved C3 1.59 mm to (29.2, 47.9)
- moved C1 1.59 mm to (21.0, 31.4)
- moved R22 1.59 mm to (24.8, 11.1)
- moved C10 1.59 mm to (21.0, 14.9)
- moved C5 1.59 mm to (21.0, 39.7)
- moved C8 1.59 mm to (21.0, 23.2)
- moved IC10 1.59 mm to (21.0, 18.1)
- moved IC2 1.59 mm to (21.0, 42.9)
- moved IC3 1.59 mm to (29.2, 42.9)
- moved IC4 1.59 mm to (21.0, 26.4)
- moved IC7 1.59 mm to (21.0, 9.84)
- moved IC9 1.59 mm to (21.0, 34.6)
- moved R12 1.59 mm to (24.8, 44.1)
- moved R18 1.59 mm to (24.8, 27.6)
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Connections:
- removed net CALL6: IC1.5
- net CELL6: now also C4.1, IC1.5
- net GND: now also C4.2
Routing:
- net CELL6: track 0.34 -> 172.8 mm
- net V1: track 0.00 -> 31.7 mm
- net CELL1: track 0.00 -> 28.9 mm
- net V2: track 0.63 -> 27.4 mm
- net V5: track 1.13 -> 27.5 mm
- net V6: track 0.00 -> 25.7 mm
- net V3: track 0.63 -> 25.0 mm
- net V4: track 0.27 -> 24.5 mm
- net CELL5: track 0.00 -> 20.0 mm
- net N$3: track 0.64 -> 20.2 mm
- net CELL2: track 0.00 -> 17.6 mm
- net N$7: track 0.78 -> 14.1 mm
- net CELL4: track 0.00 -> 13.2 mm
- net CELL3: track 0.90 -> 13.3 mm
- net N$8: track 0.64 -> 11.2 mm
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- added copper zone on layer 16, net GND

Commit message: Fix schematic
Parts:
- added CON1, CON2, CON3: 2X03, EcoCar-Connectors-2.54mm:2X03
- C1, C10, C13, C14, C2, C3, C4, C5, C8: value (none) -> 0.1
Connections:
- net CELL1: now also R20.2; no longer R19.2
- net CELL2: now also R19.2, R26.2; no longer R20.2, R25.2
- net CELL3: now also R14.2, R25.2; no longer R13.2, R26.2
- net CELL4: now also R13.2, R24.2; no longer R14.2, R23.2
- net CELL5: now also R12.2, R23.2; no longer R11.2, R24.2
- net N$1: now also R11.2; no longer R12.2
Routing:
- net CELL6: track 172.8 -> 153.9 mm
- net CELL2: track 17.6 -> 0.00 mm
- net CELL3: track 13.3 -> 0.00 mm
- net CELL4: track 13.2 -> 2.46 mm
- net N$8: track 11.2 -> 1.26 mm
- net CELL1: track 28.9 -> 22.8 mm
- net N$3: track 20.2 -> 14.6 mm
- net N$9: track 11.4 -> 6.31 mm
- net CELL5: track 20.0 -> 15.5 mm
- net N$2: track 8.16 -> 7.42 mm

Commit message: Fix routing
Parts:
- turned R14 to 180 degrees
- turned R15 to 0 degrees
- turned R16 to 0 degrees
- turned R27 to 0 degrees
Routing:
- net CELL6: track 153.9 -> 194.0 mm
- net CELL5: track 15.5 -> 51.6 mm
- net CELL2: track 0.00 -> 28.0 mm
- net CELL4: track 2.46 -> 27.3 mm
- net CELL3: track 0.00 -> 23.3 mm
- net N$1: track 5.48 -> 15.5 mm
- net CELL1: track 22.8 -> 31.5 mm
- net N$8: track 1.26 -> 9.31 mm
- net N$9: track 6.31 -> 11.4 mm
- net N$3: track 14.6 -> 19.3 mm
- net N$7: track 14.1 -> 11.2 mm
- net N$6: track 10.5 -> 9.74 mm

Commit message: More updates and gerbers
Parts:
- removed C13, C14: 0.1, EcoCar-Passives:0805
- removed IC9: AS321, AS321:AS321
- removed R25, R26, R28, R30: (no value), rcl:R0805
- added C6, C7: 0.1u, EcoCar-Passives:0805
- added CON4: 2X03, EcoCar-Connectors-2.54mm:2X03
- added IC6: AS321, AS321:AS321
- added R1: 33k, rcl:R0805
- added R2, R9: 43k, rcl:R0805
- added R4: 10k, rcl:R0805
- C1, C2, C3, C8, C9: value 0.1 -> 0.1u
- C4: value 0.1 -> 1u
- C5: value 0.1 -> 10u
- R10, R11, R12, R13, R14, R15, R16, R17, R18, R19, R20, R21, R22, R3, R5, R6, R7, R8: value (none) -> 10k
- moved IC1 41.0 mm to (21.0, 42.9)
- moved C4 37.2 mm to (3.81, 40.0), turned to 180 degrees
- moved R12 30.0 mm to (14.0, 16.2), turned to 0 degrees
- moved C1 18.5 mm to (29.2, 47.9)
- moved R17 18.0 mm to (24.8, 27.6)
- moved C5 17.3 mm to (3.81, 37.1), turned to 180 degrees
- moved C8 16.2 mm to (21.0, 6.99)
- moved R11 12.7 mm to (14.0, 23.8), turned to 0 degrees
- moved R15 12.7 mm to (14.0, 26.4), turned to 180 degrees
- moved R14 12.7 mm to (14.0, 13.7)
- moved C3 11.7 mm to (21.0, 39.7)
- moved IC3 11.7 mm to (21.0, 34.6)
- moved R7 11.1 mm to (24.8, 44.1), turned to 90 degrees
- moved IC2 8.26 mm to (29.2, 42.9)
- moved R18 8.25 mm to (24.8, 19.4)
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- renumbered C10 to C9, IC10 to IC5, R23 to R5, R24 to R8, R27 to R3, R29 to R10
Connections:
- net CELL1: now also IC7.1, R21.2; no longer IC1.1, R20.2
- net CELL2: now also R16.2, R20.2; no longer R19.2, R26.2
- net CELL3: now also R15.2; no longer R25.2
- net CELL5: now also R6.1, R7.2; no longer R12.2, R7.1
- net CELL6: now also C6.1, C7.1, IC6.5, R1.2; no longer C13.1, C14.1, IC9.5, R6.2
- net GND: now also C6.2, C7.2, IC6.2, R11.1, R12.1, R19.1, R2.1; no longer C13.2, C14.2, IC9.2, R15.1, R16.1, R21.1, R28.1
- net N$1: now also IC1.3, IC1.4, R4.2; no longer IC2.3, IC2.4, R11.2
- net N$12: now also R12.2, R14.1; no longer R25.1, R28.2
- net N$13: now also R16.1, R18.2; no longer R26.1, R30.2
- net N$15: now also IC6.1, R19.2, R20.1; no longer IC7.1, R19.1, R21.2
- net N$16: now also IC6.3, R21.1; no longer IC7.3, R20.1
- net N$2: now also IC1.1, R1.1, R6.2; no longer IC2.1, R6.1, R7.2
- net N$3: now also IC2.1, R2.2, R4.1; no longer IC3.1, R11.1, R15.2
- net N$4: now also IC2.3, R7.1, R9.2; no longer IC3.3, R12.1, R17.2
- net N$6: now also R11.2; no longer R16.2
- net N$7: now also R15.1, R17.2; no longer R14.1, R18.2
- net N$8: now also IC3.1; no longer IC9.1
- net N$9: now also IC3.3; no longer IC9.3
- net V1: now also IC7.3, IC7.4; no longer IC1.3, IC1.4
- net V2: now also IC6.4; no longer IC7.4
- net V3: now also R18.1; no longer R30.1
- net V4: now also R17.1; no longer R18.1
- net V5: now also IC3.4; no longer IC9.4
- net V6: now also IC2.4, R9.1; no longer IC3.4, R17.1
Routing:
- net CELL5: track 51.6 -> 52.4 mm
