File: cell-voltage-amplifier.sch (EAGLE design)
At the start: 44 parts, among them IC1 AS321, IC10 AS321, IC2 AS321, IC3 AS321, IC4 AS321, IC7 AS321, IC9 AS321, X1 B7B-XH-2, X2 B8B-XH-2, X3 B8B-XH-2

Commit message: Done Routing
Parts:
- added C4: (no value), EcoCar-Passives:CAPACITOR_0805
Connections:
- removed net CALL6: IC1.V+
- net CELL6: now also C4.1, IC1.V+
- net GND: now also C4.2
Changed lines of the file:
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@@
 <part name="IC1" library="AS321" deviceset="AS321" device=""/>
 <part name="X3" library="con-JST" deviceset="B8B-XH" device="-2"/>
+<part name="C4" library="EcoCar-Passives" deviceset="CAPACITOR_0805" device=""/>
 </parts>
 <sheets>
@@
 <attribute name="NAME" x="3.81" y="61.722" size="1.778" layer="95"/>
 </instance>
+<instance part="C4" gate="G$1" x="187.96" y="48.26" smashed="yes">
+<attribute name="NAME" x="189.484" y="51.181" size="1.778" layer="95" font="vector"/>
+<attribute name="VALUE" x="189.484" y="46.101" size="1.778" layer="96" font="vector"/>
+</instance>
 </instances>
 <busses>
@@
 <pinref part="X3" gate="G$1" pin="1"/>
 </segment>
+<segment>
+<pinref part="C4" gate="G$1" pin="2"/>
+<wire x1="187.96" y1="45.72" x2="185.42" y2="45.72" width="0.1524" layer="91"/>
+<label x="185.42" y="45.72" size="1.778" layer="95" rot="R180" xref="yes"/>
+</segment>
 </net>
 <net name="CELL1" class="0">
@@
 <wire x1="12.7" y1="58.42" x2="22.86" y2="58.42" width="0.1524" layer="91"/>
 <label x="22.86" y="58.42" size="1.778" layer="95" xref="yes"/>
+</segment>
+<segment>
+<pinref part="C4" gate="G$1" pin="1"/>
+<wire x1="187.96" y1="53.34" x2="185.42" y2="53.34" width="0.1524" layer="91"/>
+<label x="185.42" y="53.34" size="1.778" layer="95" rot="R180" xref="yes"/>
+</segment>
+<segment>
+<pinref part="IC1" gate="G$1" pin="V+"/>
+<wire x1="203.2" y1="68.58" x2="203.2" y2="71.12" width="0.1524" layer="91"/>
+<label x="203.2" y="71.12" size="1.778" layer="95" rot="R90" xref="yes"/>
 </segment>
 </net>
@@
 </segment>
 </net>
-<net name="CALL6" class="0">
-<segment>
-<pinref part="IC1" gate="G$1" pin="V+"/>
-<wire x1="203.2" y1="68.58" x2="203.2" y2="71.12" width="0.1524" layer="91"/>
-<label x="203.2" y="71.12" size="1.778" layer="95" rot="R90" xref="yes"/>
-</segment>
-</net>

Commit message: Fix schematic
Parts:
- added CON1, CON2, CON3: 2X03, EcoCar-Connectors-2.54mm:2X03
- C1, C10, C13, C14, C2, C3, C4, C5, C8: value (none) -> 0.1
Connections:
- net CELL1: now also R20.2; no longer R19.2
- net CELL2: now also R19.2, R26.2; no longer R20.2, R25.2
- net CELL3: now also R14.2, R25.2; no longer R13.2, R26.2
- net CELL4: now also R13.2, R24.2; no longer R14.2, R23.2
- net CELL5: now also R12.2, R23.2; no longer R11.2, R24.2
- net N$1: now also R11.2; no longer R12.2

Commit message: More updates and gerbers
Parts:
- removed C13, C14: 0.1, EcoCar-Passives:CAPACITOR_0805
- removed IC9: AS321, AS321:AS321
- removed R25, R26, R28, R30: (no value), rcl:R-US_R0805
- added C6, C7: 0.1u, EcoCar-Passives:CAPACITOR_0805
- added CON4: 2X03, EcoCar-Connectors-2.54mm:2X03
- added IC6: AS321, AS321:AS321
- added R1: 33k, rcl:R-US_R0805
- added R2, R9: 43k, rcl:R-US_R0805
- added R4: 10k, rcl:R-US_R0805
- C1, C2, C3, C8, C9: value 0.1 -> 0.1u
- C4: value 0.1 -> 1u
- C5: value 0.1 -> 10u
- R10, R11, R12, R13, R14, R15, R16, R17, R18, R19, R20, R21, R22, R3, R5, R6, R7, R8: value (none) -> 10k
- renumbered C10 to C9, IC10 to IC5, R23 to R5, R24 to R8, R27 to R3, R29 to R10
Connections:
- net CELL1: now also IC7.I+, R21.2; no longer IC1.I+, R20.2
- net CELL2: now also R16.2, R20.2; no longer R19.2, R26.2
- net CELL3: now also R15.2; no longer R25.2
- net CELL5: now also R6.1, R7.2; no longer R12.2, R7.1
- net CELL6: now also C6.1, C7.1, IC6.V+, R1.2; no longer C13.1, C14.1, IC9.V+, R6.2
- net GND: now also C6.2, C7.2, IC6.V-, R11.1, R12.1, R19.1, R2.1; no longer C13.2, C14.2, IC9.V-, R15.1, R16.1, R21.1, R28.1
- net N$1: now also IC1.I-, IC1.OUT, R4.2; no longer IC2.I-, IC2.OUT, R11.2
- net N$12: now also R12.2, R14.1; no longer R25.1, R28.2
- net N$13: now also R16.1, R18.2; no longer R26.1, R30.2
- net N$15: now also IC6.I+, R19.2, R20.1; no longer IC7.I+, R19.1, R21.2
- net N$16: now also IC6.I-, R21.1; no longer IC7.I-, R20.1
- net N$2: now also IC1.I+, R1.1, R6.2; no longer IC2.I+, R6.1, R7.2
- net N$3: now also IC2.I+, R2.2, R4.1; no longer IC3.I+, R11.1, R15.2
- net N$4: now also IC2.I-, R7.1, R9.2; no longer IC3.I-, R12.1, R17.2
- net N$6: now also R11.2; no longer R16.2
- net N$7: now also R15.1, R17.2; no longer R14.1, R18.2
- net N$8: now also IC3.I+; no longer IC9.I+
- net N$9: now also IC3.I-; no longer IC9.I-
- net V1: now also IC7.I-, IC7.OUT; no longer IC1.I-, IC1.OUT
- net V2: now also IC6.OUT; no longer IC7.OUT
- net V3: now also R18.1; no longer R30.1
- net V4: now also R17.1; no longer R18.1
- net V5: now also IC3.OUT; no longer IC9.OUT
- net V6: now also IC2.OUT, R9.1; no longer IC3.OUT, R17.1
Other:
- moved on the sheet: C1, C3, C4, C5, C8, IC1, IC2, IC3, IC7, R11, R12, R14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
