File: low-voltage-detector.brd (EAGLE design)
At the start: 50 x 50 mm, 25 parts, among them IC1 LINEAR-REGULATOR_LM317L, IC11 TL331, IC12 TL331, IC13 TL331, IC5 TL331, IC6 TL331, IC8 TL331, X1 B8B-XH-2, X2 B8B-XH-2, X3 B8B-XH-2

Commit message: saving
Parts:
- added C1, C10, C2, C3, C5, C8: (no value), EcoCar-Passives:0805
- added R3, R4, R5, R6, R7, R8: (no value), rcl:R0805
Connections:
- new net N$1: C1.1, IC5.3, R3.1
- new net N$2: C2.1, IC11.3, R4.1
- new net N$3: C3.1, IC6.3, R5.1
- new net N$4: C5.1, IC12.3, R6.1
- new net N$5: C8.1, IC8.3, R7.1
- new net N$6: C10.1, IC13.3, R8.1
- net GND: now also C1.2, C10.2, C2.2, C3.2, C5.2, C8.2
- net V1: now also R8.2; no longer IC13.3
- net V2: now also R7.2; no longer IC8.3
- net V3: now also R6.2; no longer IC12.3
- net V4: now also R5.2; no longer IC6.3
- net V5: now also R4.2; no longer IC11.3
- net V6: now also R3.2; no longer IC5.3

Commit message: Done Routing
Parts:
- added C16, C17, C18, C19, C20, C21: (no value), EcoCar-Passives:0805
- IC1: value LINEAR-REGULATOR_LM317L -> LM317L
- moved C9 8.26 mm to (28.6, 21.0)
- moved C11 8.25 mm to (28.6, 14.9)
- moved C12 8.25 mm to (28.6, 8.89)
- moved C4 8.25 mm to (28.6, 39.1)
- moved C6 8.25 mm to (28.6, 33.0)
- moved C7 8.25 mm to (28.6, 27.0)
- moved C2 1.59 mm to (20.3, 32.1)
- moved C10 1.59 mm to (20.3, 7.94)
- moved C8 1.59 mm to (20.3, 14.0)
- moved C1 1.59 mm to (20.3, 38.1)
- moved C3 1.59 mm to (20.3, 26.0)
- moved C5 1.27 mm to (20.3, 20.0)
- moved R2 0.63 mm to (12.7, 45.1)
- moved R3 0.45 mm to (13.3, 31.4)
- moved R5 0.45 mm to (13.3, 25.7)
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Connections:
- net GND: now also C16.2, C17.2, C18.2, C19.2, C20.2, C21.2
- net REF: now also C16.1, C17.1, C18.1, C19.1, C20.1, C21.1
Routing:
- net CELL6: track 0.00 -> 113.8 mm
- net REF: track 0.00 -> 71.3 mm
- net SIG1: track 0.00 -> 27.2 mm
- net SIG2: track 0.00 -> 23.7 mm
- net SIG3: track 0.00 -> 22.2 mm
- net SIG6: track 0.00 -> 22.2 mm
- net SIG4: track 0.00 -> 20.7 mm
- net SIG5: track 0.00 -> 20.7 mm
- net N$18: track 0.00 -> 15.3 mm
- net N$6: track 0.00 -> 15.3 mm
- net N$1: track 0.00 -> 11.9 mm
- net N$5: track 0.00 -> 11.9 mm
- net N$2: track 0.00 -> 10.6 mm
- net N$4: track 0.00 -> 10.6 mm
- net N$3: track 0.00 -> 10.5 mm
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- added copper zone on layer 16, net GND

Commit message: More updates and gerbers
Parts:
- removed IC8: TL331, linear:DBV-R-PDSO-G5
- added IC3: TL331, linear:DBV-R-PDSO-G5
- IC1: value LM317L -> TL331; device EcoCar-Integrated-Circuits:TO92 -> linear:DBV-R-PDSO-G5
- IC5: value TL331 -> LM317L; device linear:DBV-R-PDSO-G5 -> EcoCar-Integrated-Circuits:TO92
- R1: value TRIMPOT -> (none); device trimpot:490-2877-ND -> rcl:R0805
- R3: value (none) -> TRIMPOT; device rcl:R0805 -> trimpot:490-2877-ND
- moved C11 31.3 mm to (8.26, 38.7), turned to 180 degrees
- moved C8 29.4 mm to (4.45, 38.7)
- moved C13 28.2 mm to (28.6, 27.0), turned to 270 degrees
- moved C7 28.2 mm to (4.45, 41.6), turned to 180 degrees
- moved C15 27.0 mm to (28.6, 21.0), turned to 270 degrees
- moved C16 26.7 mm to (20.3, 14.0)
- moved C17 26.7 mm to (20.3, 7.94)
- moved C14 22.7 mm to (20.3, 22.5)
- moved C12 21.3 mm to (20.3, 28.6), turned to 180 degrees
- moved R1 17.3 mm to (13.3, 31.4), turned to 180 degrees
- moved R3 17.3 mm to (23.2, 45.7), turned to 270 degrees
- moved R2 16.5 mm to (13.3, 28.6), turned to 180 degrees
- moved R4 16.5 mm to (12.7, 45.1), turned to 0 degrees
- moved C3 14.6 mm to (20.3, 40.6)
- moved C5 14.6 mm to (20.3, 34.6)
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- renumbered IC11 to IC2, IC12 to IC4, IC13 to IC7
Connections:
- net CELL6: now also C15.1, C19.1, C21.1, C8.1, IC1.5, IC3.5, IC5.1; no longer C11.1, C12.1, C14.1, C9.1, IC1.1, IC5.5, IC8.5
- net GND: now also IC1.2, IC3.2, R3.P$3; no longer IC5.2, IC8.2, R1.P$3
- net N$1: now also IC1.3, R1.1; no longer IC5.3, R3.1
- net N$18: now also IC5.3, R3.P$2, R4.2; no longer IC1.3, R1.P$2, R2.2
- net N$2: now also R2.1; no longer R4.1
- net N$3: now also C9.1, IC3.3; no longer C3.1, IC6.3
- net N$4: now also C10.1; no longer C5.1
- net N$5: now also C16.1, IC6.3; no longer C8.1, IC8.3
- net N$6: now also C17.1; no longer C10.1
- net REF: now also C11.1, C12.1, C14.1, C3.1, C5.1, IC1.1, IC3.1, IC5.2, R4.1; no longer C15.1, C16.1, C17.1, C19.1, C21.1, IC1.2, IC5.1, IC8.1, R2.1
- net SIG2: now also IC6.4; no longer IC8.4
- net SIG4: now also IC3.4; no longer IC6.4
- net SIG6: now also IC1.4; no longer IC5.4
- net V5: now also R2.2; no longer R4.2
- net V6: now also R1.2; no longer R3.2
