File: low-voltage-detector.sch (EAGLE design)
At the start: 25 parts, among them IC1 LINEAR-REGULATOR_LM317L, IC11 TL331, IC12 TL331, IC13 TL331, IC5 TL331, IC6 TL331, IC8 TL331, X1 B8B-XH-2, X2 B8B-XH-2, X3 B8B-XH-2

Commit message: saving
Parts:
- added C1, C10, C2, C3, C5, C8: (no value), EcoCar-Passives:CAPACITOR_0805
- added R3, R4, R5, R6, R7, R8: (no value), rcl:R-US_R0805
Connections:
- new net N$1: C1.1, IC5.+IN, R3.1
- new net N$2: C2.1, IC11.+IN, R4.1
- new net N$3: C3.1, IC6.+IN, R5.1
- new net N$4: C5.1, IC12.+IN, R6.1
- new net N$5: C8.1, IC8.+IN, R7.1
- new net N$6: C10.1, IC13.+IN, R8.1
- net GND: now also C1.2, C10.2, C2.2, C3.2, C5.2, C8.2
- net V1: now also R8.2; no longer IC13.+IN
- net V2: now also R7.2; no longer IC8.+IN
- net V3: now also R6.2; no longer IC12.+IN
- net V4: now also R5.2; no longer IC6.+IN
- net V5: now also R4.2; no longer IC11.+IN
- net V6: now also R3.2; no longer IC5.+IN

Commit message: Done Routing
Parts:
- added C16, C17, C18, C19, C20, C21: (no value), EcoCar-Passives:CAPACITOR_0805
- IC1: value LINEAR-REGULATOR_LM317L -> LM317L
Connections:
- net GND: now also C16.2, C17.2, C18.2, C19.2, C20.2, C21.2
- net REF: now also C16.1, C17.1, C18.1, C19.1, C20.1, C21.1
Changed lines of the file:
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@@
 <part name="IC8" library="linear" library_urn="urn:adsk.eagle:library:262" deviceset="TL331" device="" package3d_urn="urn:adsk.eagle:package:16494/1"/>
 <part name="IC13" library="linear" library_urn="urn:adsk.eagle:library:262" deviceset="TL331" device="" package3d_urn="urn:adsk.eagle:package:16494/1"/>
-<part name="IC1" library="EcoCar-Integrated-Circuits" deviceset="LINEAR-REGULATOR_LM317L" device=""/>
+<part name="IC1" library="EcoCar-Integrated-Circuits" deviceset="LINEAR-REGULATOR_LM317L" device="" value="LM317L"/>
 <part name="R2" library="rcl" library_urn="urn:adsk.eagle:library:334" deviceset="R-US_" device="R0805" package3d_urn="urn:adsk.eagle:package:23553/2"/>
 <part name="R1" library="trimpot" deviceset="TRIMPOT" device="" package3d_urn="urn:adsk.eagle:package:3080147/2"/>
@@
 <part name="R8" library="rcl" library_urn="urn:adsk.eagle:library:334" deviceset="R-US_" device="R0805" package3d_urn="urn:adsk.eagle:package:23553/2"/>
 <part name="C10" library="EcoCar-Passives" deviceset="CAPACITOR_0805" device=""/>
+<part name="C16" library="EcoCar-Passives" deviceset="CAPACITOR_0805" device=""/>
+<part name="C17" library="EcoCar-Passives" deviceset="CAPACITOR_0805" device=""/>
+<part name="C18" library="EcoCar-Passives" deviceset="CAPACITOR_0805" device=""/>
+<part name="C19" library="EcoCar-Passives" deviceset="CAPACITOR_0805" device=""/>
+<part name="C20" library="EcoCar-Passives" deviceset="CAPACITOR_0805" device=""/>
+<part name="C21" library="EcoCar-Passives" deviceset="CAPACITOR_0805" device=""/>
 </parts>
 <sheets>
@@
 <attribute name="VALUE" x="209.296" y="70.739" size="1.778" layer="96" font="vector" rot="R180"/>
 </instance>
+<instance part="C16" gate="G$1" x="114.3" y="144.78" smashed="yes">
+<attribute name="NAME" x="115.824" y="147.701" size="1.778" layer="95" font="vector"/>
+<attribute name="VALUE" x="115.824" y="142.621" size="1.778" layer="96" font="vector"/>
+</instance>
+<instance part="C17" gate="G$1" x="203.2" y="142.24" smashed="yes">
+<attribute name="NAME" x="204.724" y="145.161" size="1.778" layer="95" font="vector"/>
+<attribute name="VALUE" x="204.724" y="140.081" size="1.778" layer="96" font="vector"/>
+</instance>
+<instance part="C18" gate="G$1" x="114.3" y="91.44" smashed="yes">
+<attribute name="NAME" x="115.824" y="94.361" size="1.778" layer="95" font="vector"/>
+<attribute name="VALUE" x="115.824" y="89.281" size="1.778" layer="96" font="vector"/>
+</instance>
+<instance part="C19" gate="G$1" x="203.2" y="91.44" smashed="yes">
+<attribute name="NAME" x="204.724" y="94.361" size="1.778" layer="95" font="vector"/>
+<attribute name="VALUE" x="204.724" y="89.281" size="1.778" layer="96" font="vector"/>
+</instance>
+<instance part="C20" gate="G$1" x="114.3" y="43.18" smashed="yes">
+<attribute name="NAME" x="115.824" y="46.101" size="1.778" layer="95" font="vector"/>
+<attribute name="VALUE" x="115.824" y="41.021" size="1.778" layer="96" font="vector"/>
+</instance>
+<instance part="C21" gate="G$1" x="200.66" y="43.18" smashed="yes">
+<attribute name="NAME" x="202.184" y="46.101" size="1.778" layer="95" font="vector"/>
+<attribute name="VALUE" x="202.184" y="41.021" size="1.778" layer="96" font="vector"/>
+</instance>
 </instances>
 <busses>
@@
 <wire x1="210.82" y1="71.12" x2="210.82" y2="73.66" width="0.1524" layer="91"/>
 <label x="210.82" y="73.66" size="1.778" layer="95" rot="R90" xref="yes"/>
+</segment>
+<segment>
+<pinref part="C16" gate="G$1" pin="2"/>
+<wire x1="114.3" y1="142.24" x2="111.76" y2="142.24" width="0.1524" layer="91"/>
+<label x="111.76" y="142.24" size="1.778" layer="95" rot="R180" xref="yes"/>
+</segment>
+<segment>
+<pinref part="C17" gate="G$1" pin="2"/>
+<wire x1="203.2" y1="139.7" x2="200.66" y2="139.7" width="0.1524" layer="91"/>
+<label x="200.66" y="139.7" size="1.778" layer="95" rot="R180" xref="yes"/>
+</segment>
+<segment>
+<pinref part="C18" gate="G$1" pin="2"/>
+<wire x1="114.3" y1="88.9" x2="111.76" y2="88.9" width="0.1524" layer="91"/>
+<label x="111.76" y="88.9" size="1.778" layer="95" rot="R180" xref="yes"/>
+</segment>
+<segment>
+<pinref part="C19" gate="G$1" pin="2"/>
+<wire x1="203.2" y1="88.9" x2="200.66" y2="88.9" width="0.1524" layer="91"/>
+<label x="200.66" y="88.9" size="1.778" layer="95" rot="R180" xref="yes"/>
+</segment>
+<segment>
+<pinref part="C20" gate="G$1" pin="2"/>
+<wire x1="114.3" y1="40.64" x2="111.76" y2="40.64" width="0.1524" layer="91"/>
+<label x="111.76" y="40.64" size="1.778" layer="95" rot="R180" xref="yes"/>
+</segment>
+<segment>
+<pinref part="C21" gate="G$1" pin="2"/>
+<wire x1="200.66" y1="40.64" x2="198.12" y2="40.64" width="0.1524" layer="91"/>
+<label x="198.12" y="40.64" size="1.778" layer="95" rot="R180" xref="yes"/>
 </segment>
 </net>
@@
 <label x="55.88" y="114.3" size="1.778" layer="95" rot="R180" xref="yes"/>
 </segment>
+<segment>
+<pinref part="C16" gate="G$1" pin="1"/>
+<wire x1="114.3" y1="149.86" x2="111.76" y2="149.86" width="0.1524" layer="91"/>
+<label x="111.76" y="149.86" size="1.778" layer="95" rot="R180" xref="yes"/>
+</segment>
+<segment>
+<pinref part="C17" gate="G$1" pin="1"/>
+<wire x1="203.2" y1="147.32" x2="200.66" y2="147.32" width="0.1524" layer="91"/>
+<label x="200.66" y="147.32" size="1.778" layer="95" rot="R180" xref="yes"/>
+</segment>
+<segment>
+<pinref part="C18" gate="G$1" pin="1"/>
+<wire x1="114.3" y1="96.52" x2="111.76" y2="96.52" width="0.1524" layer="91"/>
+<label x="111.76" y="96.52" size="1.778" layer="95" rot="R180" xref="yes"/>
+</segment>
+<segment>
+<pinref part="C19" gate="G$1" pin="1"/>
+<wire x1="203.2" y1="96.52" x2="200.66" y2="96.52" width="0.1524" layer="91"/>
+<label x="200.66" y="96.52" size="1.778" layer="95" rot="R180" xref="yes"/>
+</segment>
+<segment>
+<pinref part="C20" gate="G$1" pin="1"/>
+<wire x1="114.3" y1="48.26" x2="111.76" y2="48.26" width="0.1524" layer="91"/>
+<label x="111.76" y="48.26" size="1.778" layer="95" rot="R180" xref="yes"/>
+</segment>
+<segment>
+<pinref part="C21" gate="G$1" pin="1"/>
+<wire x1="200.66" y1="48.26" x2="198.12" y2="48.26" width="0.1524" layer="91"/>
+<label x="198.12" y="48.26" size="1.778" layer="95" rot="R180" xref="yes"/>
+</segment>
 </net>

Commit message: More updates and gerbers
Parts:
- removed IC8: TL331, linear:TL331
- added IC3: TL331, linear:TL331
- IC1: value LM317L -> TL331; device EcoCar-Integrated-Circuits:LINEAR-REGULATOR_LM317L -> linear:TL331
- IC5: value TL331 -> LM317L; device linear:TL331 -> EcoCar-Integrated-Circuits:LINEAR-REGULATOR_LM317L
- R1: value TRIMPOT -> (none); device trimpot:TRIMPOT -> rcl:R-US_R0805
- R3: value (none) -> TRIMPOT; device rcl:R-US_R0805 -> trimpot:TRIMPOT
- renumbered IC11 to IC2, IC12 to IC4, IC13 to IC7
Connections:
- net CELL6: now also C15.1, C19.1, C21.1, C8.1, IC1.V+, IC3.V+, IC5.INPUT; no longer C11.1, C12.1, C14.1, C9.1, IC1.INPUT, IC5.V+, IC8.V+
- net GND: now also IC1.GND, IC3.GND, R3.CW; no longer IC5.GND, IC8.GND, R1.CW
- net N$1: now also IC1.+IN, R1.1; no longer IC5.+IN, R3.1
- net N$18: now also IC5.ADJUST, R3.WIPER, R4.2; no longer IC1.ADJUST, R1.WIPER, R2.2
- net N$2: now also R2.1; no longer R4.1
- net N$3: now also C9.1, IC3.+IN; no longer C3.1, IC6.+IN
- net N$4: now also C10.1; no longer C5.1
- net N$5: now also C16.1, IC6.+IN; no longer C8.1, IC8.+IN
- net N$6: now also C17.1; no longer C10.1
- net REF: now also C11.1, C12.1, C14.1, C3.1, C5.1, IC1.-IN, IC3.-IN, IC5.OUTPUT, R4.1; no longer C15.1, C16.1, C17.1, C19.1, C21.1, IC1.OUTPUT, IC5.-IN, IC8.-IN, R2.1
- net SIG2: now also IC6.OUT; no longer IC8.OUT
- net SIG4: now also IC3.OUT; no longer IC6.OUT
- net SIG6: now also IC1.OUT; no longer IC5.OUT
- net V5: now also R2.2; no longer R4.2
- net V6: now also R1.2; no longer R3.2
Other:
- moved on the sheet: C10, C11, C12, C13, C14, C15, C16, C17, C18, C19, C20, C21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
