File: shutoff.brd (EAGLE design)
At the start: 50 x 50 mm, 17 parts, among them X1 B8B-XH-2

Commit message: Done Routing
Parts:
- added W1, W2, W3, W4: 16G, Wire2Board:16G
- moved D2 22.2 mm to (26.0, 32.4), turned to 90 degrees
- moved R2 12.4 mm to (21.6, 38.1)
- moved R5 8.91 mm to (9.84, 33.0), turned to 90 degrees
- moved C1 8.26 mm to (18.7, 12.1)
- moved D1 8.13 mm to (18.7, 14.6)
- moved R3 7.96 mm to (9.84, 21.9), turned to 270 degrees
- moved R1 5.97 mm to (15.9, 38.1)
- moved Q4 3.01 mm to (18.7, 27.0)
- moved R4 0.90 mm to (9.84, 27.6), turned to 270 degrees
Connections:
- removed net N$6: R3.1, R4.1, R5.1
- removed net SIG1: X1.2
- removed net SIG2: X1.3
- removed net SIG3: X1.4
- removed net SIG4: X1.5
- removed net SIG5: X1.6
- removed net SIG6: X1.7
- new net SIG: R3.1, R4.1, R5.1, X1.2, X1.3, X1.4, X1.5, X1.6, X1.7
- net BATV_E: now also W1.P$1, W4.P$1
- net BATV_I: now also W2.P$1, W3.P$1
Routing:
- net GATE: track 0.00 -> 46.7 mm
- net GND: track 0.00 -> 33.8 mm
- net SIG: track 0.00 -> 27.7 mm
- net BATV_I: track 0.00 -> 19.5 mm, vias 0 -> 22
- net N$4: track 0.00 -> 18.0 mm
- net N$3: track 0.00 -> 9.29 mm
- added copper zone on layer 1, net BATV_E
- added copper zone on layer 16, net BATV_E
- added copper zone on layer 1, net BATV_I
- added copper zone on layer 16, net BATV_I
- removed copper zone on layer 1, net GND

Commit message: More updates and gerbers
Parts:
- moved W4 34.6 mm to (21.9, 42.2), turned to 90 degrees
- moved W2 34.3 mm to (26.4, 7.94), turned to 270 degrees
- moved D1 19.2 mm to (26.0, 32.4), turned to 90 degrees
- moved D2 19.2 mm to (18.7, 14.6), turned to 0 degrees
- moved R3 11.1 mm to (9.84, 33.0), turned to 90 degrees
- moved R5 11.1 mm to (9.84, 21.9), turned to 270 degrees
- moved R1 5.71 mm to (21.6, 38.1)
- moved R2 5.71 mm to (15.9, 38.1)
- moved W3 4.45 mm to (26.4, 42.2)
Connections:
- net BATV_E: now also W2.P$1; no longer W4.P$1
- net BATV_I: now also D1.C, R1.2, R3.2, W4.P$1; no longer D2.C, R2.2, R5.2, W2.P$1
- net GATE: now also D1.A, R1.1, R2.2; no longer D2.A, R1.2, R2.1
- net GND: now also D2.A, R5.2; no longer D1.A, R3.2
- net N$3: now also R2.1; no longer R1.1
- net N$4: now also D2.C; no longer D1.C
